Commit message: Added robot_state_publisher and rviz2

File: mujoco_ros2/models/fr3_xls.urdf (robot description, URDF)
Before this commit: robot summit_xl, 28 links, 27 joints
Links:
- removed link summit_xl_base_footprint
- removed link summit_xl_base_link
- removed link v_t_link
- removed link v_x_link
- removed link v_y_link
- added link base, mass 50.455; collision mesh filename=package://mujoco_ros2/models/meshes/bases/xls/summit_xls_ch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; visual mesh filename=package://mujoco_ros2/models/meshes/bases/xls/summit_xls_ch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
- added link base_x_slide_link
- added link base_y_slide_link
- added link base_z_hinge_link
- link panda_hand: geometry visual mesh filename=package://mujoco_ros2/models/meshes/visual/hand.dae
- link panda_leftfinger: geometry visual mesh filename=package://mujoco_ros2/models/meshes/visual/finger.dae
- link panda_link0: geometry visual mesh filename=package://mujoco_ros2/models/meshes/visual/link0.dae
- link panda_link1: geometry visual mesh filename=package://mujoco_ros2/models/meshes/visual/link1.dae
- link panda_link2: geometry visual mesh filename=package://mujoco_ros2/models/meshes/visual/link2.dae
- link panda_link3: geometry visual mesh filename=package://mujoco_ros2/models/meshes/visual/link3.dae
- link panda_link4: geometry visual mesh filename=package://mujoco_ros2/models/meshes/visual/link4.dae
- link panda_link5: geometry visual mesh filename=package://mujoco_ros2/models/meshes/visual/link5.dae
- link panda_link6: geometry visual mesh filename=package://mujoco_ros2/models/meshes/visual/link6.dae
- link panda_link7: geometry visual mesh filename=package://mujoco_ros2/models/meshes/visual/link7.dae
- link panda_rightfinger: geometry visual mesh filename=package://mujoco_ros2/models/meshes/visual/finger.dae
- link summit_xl_back_left_wheel_link: geometry collision cylinder length=0.087 radius=0.127; visual mesh filename=package://mujoco_ros2/models/meshes/wheels/omni_wheel_1.dae
- link summit_xl_back_right_wheel_link: geometry collision cylinder length=0.087 radius=0.127; visual mesh filename=package://mujoco_ros2/models/meshes/wheels/omni_wheel_2.dae
- link summit_xl_base_chapa: geometry visual mesh filename=package://mujoco_ros2/models/meshes/bases/xls/summit_xls_ch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
- link summit_xl_base_logo_front: geometry visual mesh filename=package://mujoco_ros2/models/meshes/bases/xls/robotnik_logo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
- link summit_xl_base_logo_left: geometry visual mesh filename=package://mujoco_ros2/models/meshes/bases/xls/robotnik_logo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
- link summit_xl_base_logo_rear: geometry visual mesh filename=package://mujoco_ros2/models/meshes/bases/xls/robotnik_logo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
- link summit_xl_base_logo_right: geometry visual mesh filename=package://mujoco_ros2/models/meshes/bases/xls/robotnik_logo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
- link summit_xl_front_left_wheel_link: geometry collision cylinder length=0.087 radius=0.127; visual mesh filename=package://mujoco_ros2/models/meshes/wheels/omni_wheel_1.dae
- link summit_xl_front_right_wheel_link: geometry collision cylinder length=0.087 radius=0.127; visual mesh filename=package://mujoco_ros2/models/meshes/wheels/omni_wheel_2.dae
Joints:
- removed joint panda_joint1
- removed joint panda_joint2
- removed joint panda_joint3
- removed joint panda_joint4
- removed joint panda_joint5
- removed joint panda_joint6
- removed joint panda_joint7
- removed joint summit_xl_base_footprint_joint
- removed joint v_t_joint
- removed joint v_x_joint
- removed joint v_y_joint
- added joint base_x_slide_joint: type prismatic, parent base_x_slide_link, child base_y_slide_link, origin xyz=0 0 0 rpy=0 0 0, axis 1 0 0, limit lower=-10000.0 upper=-10000.0 effort=1000.0 velocity=10000.0
- added joint base_y_slide_joint: type prismatic, parent base_y_slide_link, child base_z_hinge_link, origin xyz=0 0 0 rpy=0 0 0, axis 0 1 0, limit lower=-10000.0 upper=-10000.0 effort=1000.0 velocity=10000.0
- added joint base_z_hinge_joint: type revolute, parent base_z_hinge_link, child base, origin xyz=0 0 0 rpy=0 0 0, axis 0 0 1, limit lower=-6.24 upper=6.24 effort=1000.0 velocity=10000.0
- added joint joint1: type revolute, parent panda_link0, child panda_link1, origin xyz=0 0 0.333 rpy=0 0 0, axis 0 0 1, limit lower=-2.7437 upper=2.7437 effort=87 velocity=2.1750
- added joint joint2: type revolute, parent panda_link1, child panda_link2, origin xyz=0 0 0 rpy=-1.57079632679 0 0, axis 0 0 1, limit lower=-1.7837 upper=1.7837 effort=87 velocity=2.1750
- added joint joint3: type revolute, parent panda_link2, child panda_link3, origin xyz=0 -0.316 0 rpy=1.57079632679 0 0, axis 0 0 1, limit lower=-2.9007 upper=2.9007 effort=87 velocity=2.1750
- added joint joint4: type revolute, parent panda_link3, child panda_link4, origin xyz=0.0825 0 0 rpy=1.57079632679 0 0, axis 0 0 1, limit lower=-3.0421 upper=-0.1518 effort=87 velocity=2.1750
- added joint joint5: type revolute, parent panda_link4, child panda_link5, origin xyz=-0.0825 0.384 0 rpy=-1.57079632679 0 0, axis 0 0 1, limit lower=-2.8065 upper=2.8065 effort=12 velocity=2.6100
- added joint joint6: type revolute, parent panda_link5, child panda_link6, origin xyz=0 0 0 rpy=1.57079632679 0 0, axis 0 0 1, limit lower=0.5445 upper=4.5169 effort=12 velocity=2.6100
- added joint joint7: type revolute, parent panda_link6, child panda_link7, origin xyz=0.088 0 0 rpy=1.57079632679 0 0, axis 0 0 1, limit lower=-3.0159 upper=3.0159 effort=12 velocity=2.6100
- joint panda_to_world: parent summit_xl_base_link -> base
- joint summit_xl_back_left_wheel_joint: parent summit_xl_base_link -> base
- joint summit_xl_back_right_wheel_joint: parent summit_xl_base_link -> base
- joint summit_xl_base_docking_joint: parent summit_xl_base_link -> base
- joint summit_xl_base_logo_front_joint: parent summit_xl_base_link -> base
- joint summit_xl_base_logo_left_joint: parent summit_xl_base_link -> base
- joint summit_xl_base_logo_rear_joint: parent summit_xl_base_link -> base
- joint summit_xl_base_logo_right_joint: parent summit_xl_base_link -> base
- joint summit_xl_base_tapa_joint: parent summit_xl_base_link -> base
- joint summit_xl_front_left_wheel_joint: parent summit_xl_base_link -> base
- joint summit_xl_front_right_wheel_joint: parent summit_xl_base_link -> base
- joint summit_xl_imu_joint: parent summit_xl_base_link -> base
