Commit message: inverse dynamics on joint space

File: mujoco_ros2/models/fr3.urdf (robot description, URDF)
Before this commit: robot panda, 12 links, 11 joints
Joints:
- joint panda_finger_joint1: type prismatic -> fixed
- joint panda_finger_joint2: type prismatic -> fixed

File: mujoco_ros2/models/fr3_xls_pinocchio.urdf (robot description, URDF)
Before this commit: robot summit_xl, 27 links, 26 joints
Joints:
- joint base_x_slide_joint: limit lower=-10000.0 upper=-10000.0 effort=1000.0 velocity=10000.0 -> (none); type prismatic -> fixed
- joint base_y_slide_joint: limit lower=-10000.0 upper=-10000.0 effort=1000.0 velocity=10000.0 -> (none); type prismatic -> fixed
- joint base_z_hinge_joint: limit lower=-6.24 upper=6.24 effort=1000.0 velocity=10000.0 -> (none); type revolute -> fixed
